Commit message: - Change all nodes to components - Add test cases using launch_test - Add two examples, use kuka iiwa model for testing purpose - Switch launch configuration to python -

File: models/urdf/kuka_iiwa.urdf (robot description, URDF)
Before this commit: robot kuka_iiwa, 9 links, 8 joints
Links:
- removed link kuka_lbr_l_link_0
- removed link kuka_lbr_l_link_1
- removed link kuka_lbr_l_link_2
- removed link kuka_lbr_l_link_3
- removed link kuka_lbr_l_link_4
- removed link kuka_lbr_l_link_5
- removed link kuka_lbr_l_link_6
- removed link kuka_lbr_l_link_7
- removed link kuka_lbr_l_tcp
- added link link_0, mass 5; collision mesh filename=package://wbc_ros/models/meshes/kuka_iiwa/collision/link_0_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; visual mesh filename=package://wbc_ros/models/meshes/kuka_iiwa/visual/link_0.stl
- added link link_1, mass 4; collision mesh filename=package://wbc_ros/models/meshes/kuka_iiwa/collision/link_1_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; visual mesh filename=package://wbc_ros/models/meshes/kuka_iiwa/visual/link_1.stl
- added link link_2, mass 4; collision mesh filename=package://wbc_ros/models/meshes/kuka_iiwa/collision/link_2_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; visual mesh filename=package://wbc_ros/models/meshes/kuka_iiwa/visual/link_2.stl
- added link link_3, mass 3; collision mesh filename=package://wbc_ros/models/meshes/kuka_iiwa/collision/link_3_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; visual mesh filename=package://wbc_ros/models/meshes/kuka_iiwa/visual/link_3.stl
- added link link_4, mass 2.7; collision mesh filename=package://wbc_ros/models/meshes/kuka_iiwa/collision/link_4_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; visual mesh filename=package://wbc_ros/models/meshes/kuka_iiwa/visual/link_4.stl
- added link link_5, mass 1.7; collision mesh filename=package://wbc_ros/models/meshes/kuka_iiwa/collision/link_5_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; visual mesh filename=package://wbc_ros/models/meshes/kuka_iiwa/visual/link_5.stl
- added link link_6, mass 1.8; collision mesh filename=package://wbc_ros/models/meshes/kuka_iiwa/collision/link_6_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; visual mesh filename=package://wbc_ros/models/meshes/kuka_iiwa/visual/link_6.stl
- added link link_7, mass 0.42857142857142855; collision mesh filename=package://wbc_ros/models/meshes/kuka_iiwa/collision/link_7-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; visual mesh filename=package://wbc_ros/models/meshes/kuka_iiwa/visual/link_7-MF-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
- added link link_ee
- added link world
Joints:
- removed joint kuka_lbr_l_joint_1
- removed joint kuka_lbr_l_joint_2
- removed joint kuka_lbr_l_joint_3
- removed joint kuka_lbr_l_joint_4
- removed joint kuka_lbr_l_joint_5
- removed joint kuka_lbr_l_joint_6
- removed joint kuka_lbr_l_joint_7
- removed joint kuka_lbr_l_to_tcp
- added joint joint_0: type revolute, parent link_0, child link_1, origin xyz=0 0 0.1575 rpy=0 0 0, axis 0 0 1, limit lower=-2.9670597283903604 upper=2.9670597283903604 effort=300 velocity=10
- added joint joint_1: type revolute, parent link_1, child link_2, origin xyz=0 0 0.2025 rpy=1.5707963267948966   0 3.141592653589793, axis 0 0 1, limit lower=-2.0943951023931953 upper=2.0943951023931953 effort=300 velocity=10
- added joint joint_2: type revolute, parent link_2, child link_3, origin xyz=0 0.2045 0 rpy=1.5707963267948966 0 3.141592653589793, axis 0 0 1, limit lower=-2.9670597283903604 upper=2.9670597283903604 effort=300 velocity=10
- added joint joint_3: type revolute, parent link_3, child link_4, origin xyz=0 0 0.2155 rpy=1.5707963267948966 0 0, axis 0 0 1, limit lower=-2.0943951023931953 upper=2.0943951023931953 effort=300 velocity=10
- added joint joint_4: type revolute, parent link_4, child link_5, origin xyz=0 0.1845 0 rpy=-1.5707963267948966 3.141592653589793 0, axis 0 0 1, limit lower=-2.9670597283903604 upper=2.9670597283903604 effort=300 velocity=10
- added joint joint_5: type revolute, parent link_5, child link_6, origin xyz=0 0 0.2155 rpy=1.5707963267948966 0 0, axis 0 0 1, limit lower=-2.0943951023931953 upper=2.0943951023931953 effort=300 velocity=10
- added joint joint_6: type revolute, parent link_6, child link_7, origin xyz=0 0.081 0 rpy=-1.5707963267948966 3.141592653589793 0, axis 0 0 1, limit lower=-3.0543261909900763 upper=3.0543261909900763 effort=300 velocity=10
- added joint joint_ee: type fixed, parent link_7, child link_ee, origin xyz=0 0 0.045 rpy=0 -1.5707963267948966 0
- added joint world_joint: type fixed, parent world, child link_0
